Commit message: urdf correction

File: src/robot_sim/urdf/assemblyURDF_SIM_NO_LIDAR.urdf (robot description, URDF)
Before this commit: robot quadruped_robot, 13 links, 11 joints
Joints:
- added joint leg_1_joint: type continuous, parent servo_1_link, child leg_1_link, origin xyz=0.015 -0.013 -0.00280397218834483 rpy=0 0 0.625000267634323, axis 0 0 -1
