Commit message: Update URDF file name in robot_launch.py

File: src/robot_sim/urdf/assemblyURDF_sim_v3.urdf (robot description, URDF)
Before this commit: robot quadruped_robot, 13 links, 12 joints
Links:
- link base_link: mass 0.3417 -> 0.382892713953797; geometry collision mesh filename=package://assemblyURDF_sim_v3/meshes/base_link.STL; visual mesh filename=package://assemblyURDF_sim_v3/meshes/base_link.STL
- link foot_1_link: mass 0.0046685 -> 0.00466853888839397; geometry collision mesh filename=package://assemblyURDF_sim_v3/meshes/foot_1_link.STL; visual mesh filename=package://assemblyURDF_sim_v3/meshes/foot_1_link.STL
- link foot_2_link: mass 0.0046685 -> 0.00466853888839397; geometry collision mesh filename=package://assemblyURDF_sim_v3/meshes/foot_2_link.STL; visual mesh filename=package://assemblyURDF_sim_v3/meshes/foot_2_link.STL
- link foot_3_link: mass 0.0046685 -> 0.00466853888839397; geometry collision mesh filename=package://assemblyURDF_sim_v3/meshes/foot_3_link.STL; visual mesh filename=package://assemblyURDF_sim_v3/meshes/foot_3_link.STL
- link foot_4_link: mass 0.0046685 -> 0.00466853888839397; geometry collision mesh filename=package://assemblyURDF_sim_v3/meshes/foot_4_link.STL; visual mesh filename=package://assemblyURDF_sim_v3/meshes/foot_4_link.STL
- link leg_1_link: mass 0.002267 -> 0.00226703537555513; geometry collision mesh filename=package://assemblyURDF_sim_v3/meshes/leg_1_link.STL; visual mesh filename=package://assemblyURDF_sim_v3/meshes/leg_1_link.STL
- link leg_2_link: mass 0.002267 -> 0.00226703537555513; geometry collision mesh filename=package://assemblyURDF_sim_v3/meshes/leg_2_link.STL; visual mesh filename=package://assemblyURDF_sim_v3/meshes/leg_2_link.STL
- link leg_3_link: mass 0.002267 -> 0.00226703537555514; geometry collision mesh filename=package://assemblyURDF_sim_v3/meshes/leg_3_link.STL; visual mesh filename=package://assemblyURDF_sim_v3/meshes/leg_3_link.STL
- link leg_4_link: mass 0.002267 -> 0.00226703537555514; geometry collision mesh filename=package://assemblyURDF_sim_v3/meshes/leg_4_link.STL; visual mesh filename=package://assemblyURDF_sim_v3/meshes/leg_4_link.STL
- link servo_1_link: mass 0.020716 -> 0.020715840734641; geometry collision mesh filename=package://assemblyURDF_sim_v3/meshes/servo_1_link.STL; visual mesh filename=package://assemblyURDF_sim_v3/meshes/servo_1_link.STL
- link servo_2_link: mass 0.020716 -> 0.020715840734641; geometry collision mesh filename=package://assemblyURDF_sim_v3/meshes/servo_2_link.STL; visual mesh filename=package://assemblyURDF_sim_v3/meshes/servo_2_link.STL
- link servo_3_link: mass 0.020716 -> 0.020715840734641; geometry collision mesh filename=package://assemblyURDF_sim_v3/meshes/servo_3_link.STL; visual mesh filename=package://assemblyURDF_sim_v3/meshes/servo_3_link.STL
- link servo_4_link: mass 0.020716 -> 0.020715840734641; geometry collision mesh filename=package://assemblyURDF_sim_v3/meshes/servo_4_link.STL; visual mesh filename=package://assemblyURDF_sim_v3/meshes/servo_4_link.STL
Joints:
- removed joint leg_1_joint
- joint servo_1_joint: origin xyz=0.05 -0.026 0.024 rpy=1.19325088290338 0 0 -> xyz=0.0492951218109149 -0.0235467065517865 0.024 rpy=1.19325088290338 0 0
- joint servo_2_joint: origin xyz=-0.05 -0.026 0.024 rpy=1.38644147063987 0 0 -> xyz=-0.0507048781890851 -0.0235467065517864 0.024 rpy=1.38644147063987 0 0
- joint servo_3_joint: origin xyz=-0.05 0.0259999999999996 0.0240000000000004 rpy=1.43932790895367 0 3.14159265358979 -> xyz=-0.0507048781890851 0.0284532934482131 0.0240000000000004 rpy=1.43932790895367 0 3.14159265358979
- joint servo_4_joints: origin xyz=0.05 0.0259999999999998 0.0239999999999998 rpy=1.2521204794546 0 3.14159265358979 -> xyz=0.0492951218109149 0.0284532934482133 0.0239999999999998 rpy=1.2521204794546 0 3.14159265358979
