Commit message: Update robot model meshes (MODEL WITHOUT LIDAR DISPLAYING)

File: src/robot_model/urdf/assemblyURDF_sim_v3.urdf (robot description, URDF)
Before this commit: robot assemblyURDF_sim_v3, 13 links, 11 joints
Links:
- link base_link: mass 0.382892713953797 -> 0.3417
- link foot_1_link: mass 0.00466853888839397 -> 0.0046685
- link foot_2_link: mass 0.00466853888839397 -> 0.0046685
- link foot_3_link: mass 0.00466853888839397 -> 0.0046685
- link foot_4_link: mass 0.00466853888839397 -> 0.0046685
- link leg_1_link: mass 0.00226703537555513 -> 0.002267
- link leg_2_link: mass 0.00226703537555513 -> 0.002267
- link leg_3_link: mass 0.00226703537555514 -> 0.002267
- link leg_4_link: mass 0.00226703537555514 -> 0.002267
- link servo_1_link: mass 0.020715840734641 -> 0.020716
- link servo_2_link: mass 0.020715840734641 -> 0.020716
- link servo_3_link: mass 0.020715840734641 -> 0.020716
- link servo_4_link: mass 0.020715840734641 -> 0.020716
Joints:
- added joint leg_1_joint: type continuous, parent servo_1_link, child leg_1_link, origin xyz=0.015 -0.013 -0.00280397218834483 rpy=0 0 0.625000267634323, axis 0 0 -1
- joint servo_1_joint: origin xyz=0.0492951218109149 -0.0235467065517865 0.024 rpy=1.19325088290338 0 0 -> xyz=0.05 -0.026 0.024 rpy=1.19325088290338 0 0
- joint servo_2_joint: origin xyz=-0.0507048781890851 -0.0235467065517864 0.024 rpy=1.38644147063987 0 0 -> xyz=-0.05 -0.026 0.024 rpy=1.38644147063987 0 0
- joint servo_3_joint: origin xyz=-0.0507048781890851 0.0284532934482131 0.0240000000000004 rpy=1.43932790895367 0 3.14159265358979 -> xyz=-0.05 0.0259999999999996 0.0240000000000004 rpy=1.43932790895367 0 3.14159265358979
- joint servo_4_joints: origin xyz=0.0492951218109149 0.0284532934482133 0.0239999999999998 rpy=1.2521204794546 0 3.14159265358979 -> xyz=0.05 0.0259999999999998 0.0239999999999998 rpy=1.2521204794546 0 3.14159265358979

Commit message: Update robot model  files (LIDAR VERSION DISPLAYING)

File: src/robot_model/urdf/assemblyURDF_sim_v3.urdf (robot description, URDF)
Before this commit: robot assemblyURDF_sim_v3, 13 links, 12 joints
Links:
- link base_link: mass 0.3417 -> 0.382892713953797
- link foot_1_link: mass 0.0046685 -> 0.00466853888839397
- link foot_2_link: mass 0.0046685 -> 0.00466853888839397
- link foot_3_link: mass 0.0046685 -> 0.00466853888839397
- link foot_4_link: mass 0.0046685 -> 0.00466853888839397
- link leg_1_link: mass 0.002267 -> 0.00226703537555513
- link leg_2_link: mass 0.002267 -> 0.00226703537555513
- link leg_3_link: mass 0.002267 -> 0.00226703537555514
- link leg_4_link: mass 0.002267 -> 0.00226703537555514
- link servo_1_link: mass 0.020716 -> 0.020715840734641
- link servo_2_link: mass 0.020716 -> 0.020715840734641
- link servo_3_link: mass 0.020716 -> 0.020715840734641
- link servo_4_link: mass 0.020716 -> 0.020715840734641
Joints:
- joint servo_1_joint: origin xyz=0.05 -0.026 0.024 rpy=1.19325088290338 0 0 -> xyz=0.0492951218109149 -0.0235467065517865 0.024 rpy=1.19325088290338 0 0
- joint servo_2_joint: origin xyz=-0.05 -0.026 0.024 rpy=1.38644147063987 0 0 -> xyz=-0.0507048781890851 -0.0235467065517864 0.024 rpy=1.38644147063987 0 0
- joint servo_3_joint: origin xyz=-0.05 0.0259999999999996 0.0240000000000004 rpy=1.43932790895367 0 3.14159265358979 -> xyz=-0.0507048781890851 0.0284532934482131 0.0240000000000004 rpy=1.43932790895367 0 3.14159265358979
- joint servo_4_joints: origin xyz=0.05 0.0259999999999998 0.0239999999999998 rpy=1.2521204794546 0 3.14159265358979 -> xyz=0.0492951218109149 0.0284532934482133 0.0239999999999998 rpy=1.2521204794546 0 3.14159265358979
